File: NixieClock/MainClock.sch (EAGLE design)
At the start: 87 parts, among them IC1 MEGA8-P, IC2 74141N, IC3 NE555, Q1 MPSA 42, Q10 IRF740, Q11 BC547, Q12 MPSA 92, Q13 MPSA 42, Q14 MPSA 42, Q15 MPSA55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

Commit message: Moved Names and Values so that they are easily readable
Parts:
- renumbered 9V/12-35V-DC-IN to 9V/12-35V
Changed lines of the file:
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@@
 <part name="BUZZER" library="buzzer" library_urn="urn:adsk.eagle:library:113" deviceset="F/TMB" device="" package3d_urn="urn:adsk.eagle:package:5260/1"/>
 <part name="R34" library="resistor" library_urn="urn:adsk.eagle:library:348" deviceset="R-EU_" device="0411/15" package3d_urn="urn:adsk.eagle:package:26093/1" value="100 Ohm"/>
-<part name="9V/12-35V-DC-IN" library="con-jack" library_urn="urn:adsk.eagle:library:154" deviceset="JACK-PLUG" device="1" package3d_urn="urn:adsk.eagle:package:7494/1"/>
+<part name="9V/12-35V" library="con-jack" library_urn="urn:adsk.eagle:library:154" deviceset="JACK-PLUG" device="1" package3d_urn="urn:adsk.eagle:package:7494/1"/>
 <part name="GND2" library="supply1" library_urn="urn:adsk.eagle:library:371" deviceset="GND" device=""/>
 <part name="D4" library="diode" library_urn="urn:adsk.eagle:library:210" deviceset="1N4004" device="" package3d_urn="urn:adsk.eagle:package:43336/1"/>
@@
 <instance part="BUZZER" gate="1" x="-43.18" y="55.88" rot="R270"/>
 <instance part="R34" gate="G$1" x="-27.94" y="60.96" rot="R180"/>
-<instance part="9V/12-35V-DC-IN" gate="G$1" x="0" y="143"/>
+<instance part="9V/12-35V" gate="G$1" x="0" y="143"/>
 <instance part="GND2" gate="1" x="13" y="132"/>
 <instance part="D4" gate="1" x="27.94" y="144.78"/>
@@
 </segment>
 <segment>
-<pinref part="9V/12-35V-DC-IN" gate="G$1" pin="1"/>
+<pinref part="9V/12-35V" gate="G$1" pin="1"/>
 <pinref part="GND2" gate="1" pin="GND"/>
 <wire x1="13" y1="134.54" x2="13" y2="140" width="0.1524" layer="91"/>
 <wire x1="13" y1="140" x2="8" y2="140" width="0.1524" layer="91"/>
-<pinref part="9V/12-35V-DC-IN" gate="G$1" pin="2"/>
+<pinref part="9V/12-35V" gate="G$1" pin="2"/>
 <wire x1="8" y1="140" x2="5.08" y2="140.46" width="0.1524" layer="91"/>
 <wire x1="5.08" y1="143" x2="8" y2="143" width="0.1524" layer="91"/>
@@
 <net name="N$5" class="0">
 <segment>
-<pinref part="9V/12-35V-DC-IN" gate="G$1" pin="3"/>
+<pinref part="9V/12-35V" gate="G$1" pin="3"/>
 <pinref part="D4" gate="1" pin="A"/>
 <wire x1="5.08" y1="145.54" x2="25.4" y2="144.78" width="0.1524" layer="91"/>

Commit message: Added a button to the board and added the shield
Parts:
- added CATHODDETOX: (no value), switch-omron:31-XX
Connections:
- new net ANALOG_2: CATHODDETOX.P, IC1.PC2(ADC2)
- net GND: now also CATHODDETOX.S
Changed lines of the file:
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@@
 <setting verticaltext="up"/>
 </settings>
-<grid distance="0.1" unitdist="inch" unit="inch" style="lines" multiple="1" display="no" altdistance="0.01" altunitdist="inch" altunit="inch"/>
+<grid distance="1" unitdist="mm" unit="mm" style="lines" multiple="1" display="no" altdistance="1" altunitdist="mm" altunit="mm"/>
 <layers>
 <layer number="1" name="Top" color="4" fill="1" visible="no" active="no"/>
@@
 <part name="L7809" library="v-reg" library_urn="urn:adsk.eagle:library:409" deviceset="78XXS" device="" package3d_urn="urn:adsk.eagle:package:30342/1"/>
 <part name="L7805CV" library="v-reg" library_urn="urn:adsk.eagle:library:409" deviceset="78XXS" device="" package3d_urn="urn:adsk.eagle:package:30342/1"/>
+<part name="CATHODDETOX" library="switch-omron" library_urn="urn:adsk.eagle:library:377" deviceset="31-XX" device="" package3d_urn="urn:adsk.eagle:package:27487/1"/>
+<part name="GND22" library="supply1" library_urn="urn:adsk.eagle:library:371" deviceset="GND" device=""/>
 </parts>
 <sheets>
@@
 <wire x1="0.38" y1="157" x2="0.38" y2="157.48" width="0.1524" layer="91"/>
 <wire x1="0.38" y1="157.48" x2="-5.08" y2="157.48" width="0.1524" layer="91"/>
+</segment>
+</net>
+<net name="ANALOG_2" class="0">
+<segment>
+<pinref part="IC1" gate="G$1" pin="PC2(ADC2)"/>
+<wire x1="33.02" y1="99.06" x2="38.1" y2="99.06" width="0.1524" layer="91"/>
+<label x="33.02" y="99.06" size="1.778" layer="95"/>
 </segment>
 </net>
@@
 <instance part="GND21" gate="1" x="210.82" y="17.78"/>
 <instance part="+180V(TEST)" gate="G$1" x="213" y="131"/>
+<instance part="CATHODDETOX" gate="1" x="352" y="156" rot="R270"/>
+<instance part="GND22" gate="1" x="360" y="139"/>
 </instances>
 <busses>
@@
 <pinref part="GND20" gate="1" pin="GND"/>
 <wire x1="241.3" y1="20.32" x2="241.3" y2="15.24" width="0.1524" layer="91"/>
+</segment>
+<segment>
+<pinref part="CATHODDETOX" gate="1" pin="S"/>
+<pinref part="GND22" gate="1" pin="GND"/>
+<wire x1="357.08" y1="156" x2="360" y2="156" width="0.1524" layer="91"/>
+<wire x1="360" y1="156" x2="360" y2="141.54" width="0.1524" layer="91"/>
 </segment>
 </net>
@@
 </segment>
 </net>
+<net name="ANALOG_2" class="0">
+<segment>
+<pinref part="CATHODDETOX" gate="1" pin="P"/>
+<wire x1="346.92" y1="156" x2="340.36" y2="156" width="0.1524" layer="91"/>
+<wire x1="340.36" y1="156" x2="340.36" y2="157.48" width="0.1524" layer="91"/>
+<label x="335" y="156" size="1.778" layer="95"/>
+</segment>
+</net>
